File: VesselV2.kicad_pcb (KiCad board)
At the start: 2 copper layers, 209 parts, among them U1 ATmega32U4-A

Commit message: Pcb build done - Adding crystal & labels
Parts:
- removed S4: MX_stab, PCM_marbastlib-mx:STAB_MX_P_6.25u
- D1, D10, D100, D101, D102, D11, D12, D13, D14, D15, D16, D17, D18, D19, D2, D20, D21, D22, D23, D24, D25, D26, D27, D28, D29, D3, D30, D31, D32, D33, D34, D35, D36, D37, D38, D39, D4, D40, D41, D42, D43, D44, D45, D46, D47, D48, D49, D5, D50, D51, D52, D53, D54, D55, D56, D57, D58, D59, D6, D60, D61, D62, D63, D64, D65, D66, D67, D68, D69, D7, D70, D71, D72, D73, D74, D75, D76, D77, D78, D79, D8, D80, D81, D82, D83, D84, D85, D86, D87, D88, D89, D9, D90, D91, D92, D93, D94, D95, D96, D97, D98, D99: moved to B.Cu
- MX91: footprint PCM_marbastlib-mx:SW_MX_1u -> PCM_marbastlib-mx:SW_MX_1.75u
- S3: footprint PCM_marbastlib-mx:STAB_MX_P_2u -> PCM_marbastlib-mx:STAB_MX_P_6.25u
- moved MX48 786.4 mm to (109.5, 152.4)
- moved D94 782.8 mm to (110.3, 210.3), turned to 90 degrees
- moved D79 778.7 mm to (110.3, 191.3), turned to 90 degrees
- moved D32 770.5 mm to (108.0, 134.1), turned to 90 degrees
- moved D64 770.3 mm to (115.1, 172.2), turned to 90 degrees
- moved D48 769.1 mm to (112.7, 153.2), turned to 90 degrees
- moved D16 768.5 mm to (108.0, 110.3), turned to 90 degrees
- moved D1 767.8 mm to (108.0, 86.5), turned to 90 degrees
- moved MX79 766.0 mm to (107.2, 190.5)
- moved MX94 765.8 mm to (107.2, 209.6)
- moved D95 759.3 mm to (134.1, 210.3), turned to 90 degrees
- moved D80 757.7 mm to (131.8, 191.3), turned to 90 degrees
- moved D33 752.3 mm to (127.0, 134.1), turned to 90 degrees
- moved D2 750.0 mm to (127.0, 86.5), turned to 90 degrees
- moved D49 746.0 mm to (136.5, 153.2), turned to 90 degrees
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
Commit message: Edge cuts done - Datasheet info filled in - Preliminary Bom generated
Parts:
- added ?: ?, PCBPersonalLogos:VesselLogoPCB, F.Cu at (421.5, 210.3)
- added C1: 22pF, Capacitor_SMD:C_0805_2012Metric_Pad1.18x1.45mm_HandSolder, F.Cu at (410.8, 52.4)
- added C2: 1uf, Capacitor_SMD:C_0805_2012Metric_Pad1.18x1.45mm_HandSolder, B.Cu at (410.4, 68.1)
- added C3: 22pF, Capacitor_SMD:C_0805_2012Metric_Pad1.18x1.45mm_HandSolder, F.Cu at (417.2, 58.5)
- added F1: 500mA, Fuse:Fuse_1206_3216Metric_Pad1.42x1.75mm_HandSolder, B.Cu at (272.3, 51.8)
- added R2: 22, Resistor_SMD:R_0805_2012Metric_Pad1.20x1.40mm_HandSolder, F.Cu at (411.2, 73.7)
- added R3: 22, Resistor_SMD:R_0805_2012Metric_Pad1.20x1.40mm_HandSolder, F.Cu at (409.6, 72.1)
- added R4: 10k, Resistor_SMD:R_0805_2012Metric_Pad1.20x1.40mm_HandSolder, F.Cu at (417.3, 67.5)
- added R5: 10k, Resistor_SMD:R_0805_2012Metric_Pad1.20x1.40mm_HandSolder, F.Cu at (392.8, 61.9)
- added SW1: SW_Push, random-keyboard-parts:SKQG-1155865, F.Cu at (421.3, 63.5)
- added USB1: Molex-0548190589, random-keyboard-parts:Molex-0548190589, F.Cu at (263.5, 49.5)
- added Y1: 16MHz, Crystal:Crystal_SMD_3225-4Pin_3.2x2.5mm_HandSoldering, F.Cu at (413.9, 55.8)
- moved U1 14.0 mm to (404.8, 61.9)
Connections:
- D1 pad 1: Net-(D1-K) -> ROW0
- D10 pad 1: Net-(D1-K) -> ROW0
- D100 pad 1: Net-(D100-K) -> ROW6
- D101 pad 1: Net-(D100-K) -> ROW6
- D102 pad 1: Net-(D100-K) -> ROW6
- D11 pad 1: Net-(D1-K) -> ROW0
- D12 pad 1: Net-(D1-K) -> ROW0
- D13 pad 1: Net-(D1-K) -> ROW0
- D14 pad 1: Net-(D1-K) -> ROW0
- D15 pad 1: Net-(D1-K) -> ROW0
- D16 pad 1: Net-(D16-K) -> ROW1
- D17 pad 1: Net-(D16-K) -> ROW1
- D18 pad 1: Net-(D16-K) -> ROW1
- D19 pad 1: Net-(D16-K) -> ROW1
- D2 pad 1: Net-(D1-K) -> ROW0
- D20 pad 1: Net-(D16-K) -> ROW1
- D21 pad 1: Net-(D16-K) -> ROW1
- D22 pad 1: Net-(D16-K) -> ROW1
- D23 pad 1: Net-(D16-K) -> ROW1
- D24 pad 1: Net-(D16-K) -> ROW1
- D25 pad 1: Net-(D16-K) -> ROW1
- D26 pad 1: Net-(D16-K) -> ROW1
- D27 pad 1: Net-(D16-K) -> ROW1
- D28 pad 1: Net-(D16-K) -> ROW1
- D29 pad 1: Net-(D16-K) -> ROW1
- D3 pad 1: Net-(D1-K) -> ROW0
- D30 pad 1: Net-(D16-K) -> ROW1
- D31 pad 1: Net-(D16-K) -> ROW1
- D32 pad 1: Net-(D32-K) -> ROW2
- D33 pad 1: Net-(D32-K) -> ROW2
- D34 pad 1: Net-(D32-K) -> ROW2
- D35 pad 1: Net-(D32-K) -> ROW2
- D36 pad 1: Net-(D32-K) -> ROW2
- D37 pad 1: Net-(D32-K) -> ROW2
- D38 pad 1: Net-(D32-K) -> ROW2
- D39 pad 1: Net-(D32-K) -> ROW2
- D4 pad 1: Net-(D1-K) -> ROW0
- D40 pad 1: Net-(D32-K) -> ROW2
- D41 pad 1: Net-(D32-K) -> ROW2
- D42 pad 1: Net-(D32-K) -> ROW2
- D43 pad 1: Net-(D32-K) -> ROW2
- D44 pad 1: Net-(D32-K) -> ROW2
- D45 pad 1: Net-(D32-K) -> ROW2
- D46 pad 1: Net-(D32-K) -> ROW2
- D47 pad 1: Net-(D32-K) -> ROW2
- D48 pad 1: Net-(D48-K) -> ROW3
- D49 pad 1: Net-(D48-K) -> ROW3
- D5 pad 1: Net-(D1-K) -> ROW0
- D50 pad 1: Net-(D48-K) -> ROW3
- D51 pad 1: Net-(D48-K) -> ROW3
- D52 pad 1: Net-(D48-K) -> ROW3
- D53 pad 1: Net-(D48-K) -> ROW3
- D54 pad 1: Net-(D48-K) -> ROW3
- D55 pad 1: Net-(D48-K) -> ROW3
- D56 pad 1: Net-(D48-K) -> ROW3
- D57 pad 1: Net-(D48-K) -> ROW3
- D58 pad 1: Net-(D48-K) -> ROW3
- D59 pad 1: Net-(D48-K) -> ROW3
- D6 pad 1: Net-(D1-K) -> ROW0
- D60 pad 1: Net-(D48-K) -> ROW3
- D61 pad 1: Net-(D48-K) -> ROW3
- D62 pad 1: Net-(D48-K) -> ROW3
- D63 pad 1: Net-(D48-K) -> ROW3
- D64 pad 1: Net-(D64-K) -> ROW4
- D65 pad 1: Net-(D64-K) -> ROW4
- D66 pad 1: Net-(D64-K) -> ROW4
- D67 pad 1: Net-(D64-K) -> ROW4
- D68 pad 1: Net-(D64-K) -> ROW4
- D69 pad 1: Net-(D64-K) -> ROW4
- D7 pad 1: Net-(D1-K) -> ROW0
- D70 pad 1: Net-(D64-K) -> ROW4
- D71 pad 1: Net-(D64-K) -> ROW4
- D72 pad 1: Net-(D64-K) -> ROW4
- D73 pad 1: Net-(D64-K) -> ROW4
- D74 pad 1: Net-(D64-K) -> ROW4
- D75 pad 1: Net-(D64-K) -> ROW4
- D76 pad 1: Net-(D64-K) -> ROW4
- D77 pad 1: Net-(D64-K) -> ROW4
- D78 pad 1: Net-(D64-K) -> ROW4
- D79 pad 1: Net-(D79-K) -> ROW5
- D8 pad 1: Net-(D1-K) -> ROW0
- D80 pad 1: Net-(D79-K) -> ROW5
- D81 pad 1: Net-(D79-K) -> ROW5
- D82 pad 1: Net-(D79-K) -> ROW5
- D83 pad 1: Net-(D79-K) -> ROW5
- D84 pad 1: Net-(D79-K) -> ROW5
- D85 pad 1: Net-(D79-K) -> ROW5
- D86 pad 1: Net-(D79-K) -> ROW5
- D87 pad 1: Net-(D79-K) -> ROW5
- D88 pad 1: Net-(D79-K) -> ROW5
- D89 pad 1: Net-(D79-K) -> ROW5
- D9 pad 1: Net-(D1-K) -> ROW0
- D90 pad 1: Net-(D79-K) -> ROW5
- D91 pad 1: Net-(D79-K) -> ROW5
- D92 pad 1: Net-(D79-K) -> ROW5
- D93 pad 1: Net-(D79-K) -> ROW5
- D94 pad 1: Net-(D100-K) -> ROW6
- D95 pad 1: Net-(D100-K) -> ROW6
- D96 pad 1: Net-(D100-K) -> ROW6
- D97 pad 1: Net-(D100-K) -> ROW6
- D98 pad 1: Net-(D100-K) -> ROW6
- D99 pad 1: Net-(D100-K) -> ROW6
- MX1 pad 1: Net-(MX1-Pad1) -> COL0
- MX10 pad 1: Net-(MX10-Pad1) -> COL10
- MX100 pad 1: Net-(MX100-Pad1) -> COL12
- MX101 pad 1: Net-(MX101-Pad1) -> COL13
- MX102 pad 1: Net-(MX102-Pad1) -> COL14
- MX11 pad 1: Net-(MX11-Pad1) -> COL11
- MX12 pad 1: Net-(MX100-Pad1) -> COL12
- MX13 pad 1: Net-(MX102-Pad1) -> COL14
- MX14 pad 1: Net-(MX14-Pad1) -> COL15
- MX15 pad 1: Net-(MX15-Pad1) -> COL16
- MX16 pad 1: Net-(MX1-Pad1) -> COL0
- MX17 pad 1: Net-(MX17-Pad1) -> COL2
- MX18 pad 1: Net-(MX18-Pad1) -> COL3
- MX19 pad 1: Net-(MX19-Pad1) -> COL4
- MX2 pad 1: Net-(MX2-Pad1) -> COL1
- MX20 pad 1: Net-(MX20-Pad1) -> COL5
- MX21 pad 1: Net-(MX21-Pad1) -> COL6
- MX22 pad 1: Net-(MX22-Pad1) -> COL7
- MX23 pad 1: Net-(MX23-Pad1) -> COL9
- MX24 pad 1: Net-(MX24-Pad1) -> COL8
- MX25 pad 1: Net-(MX10-Pad1) -> COL10
- MX26 pad 1: Net-(MX11-Pad1) -> COL11
- MX27 pad 1: Net-(MX100-Pad1) -> COL12
- MX28 pad 1: Net-(MX101-Pad1) -> COL13
- MX29 pad 1: Net-(MX102-Pad1) -> COL14
- MX3 pad 1: Net-(MX17-Pad1) -> COL2
- MX30 pad 1: Net-(MX14-Pad1) -> COL15
- MX31 pad 1: Net-(MX15-Pad1) -> COL16
- MX32 pad 1: Net-(MX1-Pad1) -> COL0
- MX33 pad 1: Net-(MX2-Pad1) -> COL1
- MX34 pad 1: Net-(MX17-Pad1) -> COL2
- MX35 pad 1: Net-(MX18-Pad1) -> COL3
- MX36 pad 1: Net-(MX19-Pad1) -> COL4
- MX37 pad 1: Net-(MX20-Pad1) -> COL5
- MX38 pad 1: Net-(MX21-Pad1) -> COL6
- MX39 pad 1: Net-(MX22-Pad1) -> COL7
- MX4 pad 1: Net-(MX18-Pad1) -> COL3
- MX40 pad 1: Net-(MX23-Pad1) -> COL9
- MX41 pad 1: Net-(MX24-Pad1) -> COL8
- MX42 pad 1: Net-(MX10-Pad1) -> COL10
- MX43 pad 1: Net-(MX11-Pad1) -> COL11
- MX44 pad 1: Net-(MX100-Pad1) -> COL12
- MX45 pad 1: Net-(MX101-Pad1) -> COL13
- MX46 pad 1: Net-(MX14-Pad1) -> COL15
- MX47 pad 1: Net-(MX15-Pad1) -> COL16
- MX48 pad 1: Net-(MX1-Pad1) -> COL0
- MX49 pad 1: Net-(MX2-Pad1) -> COL1
- MX5 pad 1: Net-(MX19-Pad1) -> COL4
- MX50 pad 1: Net-(MX17-Pad1) -> COL2
- MX51 pad 1: Net-(MX18-Pad1) -> COL3
- MX52 pad 1: Net-(MX19-Pad1) -> COL4
- MX53 pad 1: Net-(MX20-Pad1) -> COL5
- MX54 pad 1: Net-(MX21-Pad1) -> COL6
- MX55 pad 1: Net-(MX22-Pad1) -> COL7
- MX56 pad 1: Net-(MX23-Pad1) -> COL9
- MX57 pad 1: Net-(MX24-Pad1) -> COL8
- MX58 pad 1: Net-(MX10-Pad1) -> COL10
- MX59 pad 1: Net-(MX11-Pad1) -> COL11
- MX6 pad 1: Net-(MX20-Pad1) -> COL5
- MX60 pad 1: Net-(MX100-Pad1) -> COL12
- MX61 pad 1: Net-(MX101-Pad1) -> COL13
- MX62 pad 1: Net-(MX14-Pad1) -> COL15
- MX63 pad 1: Net-(MX15-Pad1) -> COL16
- MX64 pad 1: Net-(MX1-Pad1) -> COL0
- MX65 pad 1: Net-(MX2-Pad1) -> COL1
- MX66 pad 1: Net-(MX17-Pad1) -> COL2
- MX67 pad 1: Net-(MX18-Pad1) -> COL3
- MX68 pad 1: Net-(MX19-Pad1) -> COL4
- MX69 pad 1: Net-(MX20-Pad1) -> COL5
- MX7 pad 1: Net-(MX21-Pad1) -> COL6
- MX70 pad 1: Net-(MX21-Pad1) -> COL6
- MX71 pad 1: Net-(MX22-Pad1) -> COL7
- MX72 pad 1: Net-(MX23-Pad1) -> COL9
- MX73 pad 1: Net-(MX24-Pad1) -> COL8
- MX74 pad 1: Net-(MX10-Pad1) -> COL10
- MX75 pad 1: Net-(MX11-Pad1) -> COL11
- MX76 pad 1: Net-(MX100-Pad1) -> COL12
- MX77 pad 1: Net-(MX14-Pad1) -> COL15
- MX78 pad 1: Net-(MX15-Pad1) -> COL16
- MX79 pad 1: Net-(MX1-Pad1) -> COL0
- MX8 pad 1: Net-(MX22-Pad1) -> COL7
- MX80 pad 1: Net-(MX2-Pad1) -> COL1
- MX81 pad 1: Net-(MX17-Pad1) -> COL2
- MX82 pad 1: Net-(MX18-Pad1) -> COL3
- MX83 pad 1: Net-(MX19-Pad1) -> COL4
- MX84 pad 1: Net-(MX20-Pad1) -> COL5
- MX85 pad 1: Net-(MX21-Pad1) -> COL6
- MX86 pad 1: Net-(MX22-Pad1) -> COL7
- MX87 pad 1: Net-(MX23-Pad1) -> COL9
- MX88 pad 1: Net-(MX24-Pad1) -> COL8
- MX89 pad 1: Net-(MX10-Pad1) -> COL10
- MX9 pad 1: Net-(MX23-Pad1) -> COL9
- MX90 pad 1: Net-(MX11-Pad1) -> COL11
- MX91 pad 1: Net-(MX100-Pad1) -> COL12
- MX92 pad 1: Net-(MX101-Pad1) -> COL13
- MX93 pad 1: Net-(MX15-Pad1) -> COL16
- MX94 pad 1: Net-(MX1-Pad1) -> COL0
- MX95 pad 1: Net-(MX2-Pad1) -> COL1
- MX96 pad 1: Net-(MX17-Pad1) -> COL2
- MX97 pad 1: Net-(MX21-Pad1) -> COL6
- MX98 pad 1: Net-(MX24-Pad1) -> COL8
- MX99 pad 1: Net-(MX10-Pad1) -> COL10
- U1 pad 10: unconnected-(U1-PB2-Pad10) -> ROW2
- U1 pad 11: unconnected-(U1-PB3-Pad11) -> ROW3
- U1 pad 12: unconnected-(U1-PB7-Pad12) -> COL0
- U1 pad 13: unconnected-(U1-~{RESET}-Pad13) -> Net-(U1-~{RESET})
- U1 pad 14: Net-(U1-VCC-Pad14) -> +5V
- U1 pad 15: Net-(U1-GND-Pad15) -> GND
- U1 pad 16: unconnected-(U1-XTAL2-Pad16) -> Net-(U1-XTAL2)
- U1 pad 17: unconnected-(U1-XTAL1-Pad17) -> Net-(U1-XTAL1)
- U1 pad 18: unconnected-(U1-PD0-Pad18) -> ROW4
- U1 pad 19: unconnected-(U1-PD1-Pad19) -> ROW5
- U1 pad 2: unconnected-(U1-UVCC-Pad2) -> +5V
- U1 pad 20: unconnected-(U1-PD2-Pad20) -> ROW6
- U1 pad 21: unconnected-(U1-PD3-Pad21) -> COL1
- U1 pad 22: unconnected-(U1-PD5-Pad22) -> COL2
- U1 pad 23: Net-(U1-GND-Pad15) -> GND
- U1 pad 24: Net-(U1-AVCC-Pad24) -> +5V
- U1 pad 25: unconnected-(U1-PD4-Pad25) -> COL3
- U1 pad 26: unconnected-(U1-PD6-Pad26) -> COL4
- U1 pad 27: unconnected-(U1-PD7-Pad27) -> COL5
- U1 pad 28: unconnected-(U1-PB4-Pad28) -> COL6
- U1 pad 29: unconnected-(U1-PB5-Pad29) -> COL7
- U1 pad 3: unconnected-(U1-D--Pad3) -> Net-(U1-D-)
- U1 pad 30: unconnected-(U1-PB6-Pad30) -> COL8
- U1 pad 31: unconnected-(U1-PC6-Pad31) -> COL9
- U1 pad 32: unconnected-(U1-PC7-Pad32) -> COL10
- U1 pad 33: unconnected-(U1-~{HWB}/PE2-Pad33) -> Net-(U1-~{HWB}/PE2)
- U1 pad 34: Net-(U1-VCC-Pad14) -> +5V
- U1 pad 35: Net-(U1-GND-Pad15) -> GND
- U1 pad 36: unconnected-(U1-PF7-Pad36) -> COL11
- U1 pad 37: unconnected-(U1-PF6-Pad37) -> COL12
- U1 pad 38: unconnected-(U1-PF5-Pad38) -> COL13
- U1 pad 39: unconnected-(U1-PF4-Pad39) -> COL14
- U1 pad 4: unconnected-(U1-D+-Pad4) -> Net-(U1-D+)
- U1 pad 40: unconnected-(U1-PF1-Pad40) -> COL15
- U1 pad 41: unconnected-(U1-PF0-Pad41) -> COL16
- U1 pad 43: Net-(U1-GND-Pad15) -> GND
- U1 pad 44: Net-(U1-AVCC-Pad24) -> +5V
- U1 pad 5: unconnected-(U1-UGND-Pad5) -> GND
- U1 pad 6: unconnected-(U1-UCAP-Pad6) -> Net-(U1-UCAP)
- U1 pad 7: unconnected-(U1-VBUS-Pad7) -> +5V
- U1 pad 8: unconnected-(U1-PB0-Pad8) -> ROW0
- U1 pad 9: unconnected-(U1-PB1-Pad9) -> ROW1
Other:
- board outline added: 345.3 x 176.2 mm
- board text added: "Vessel - Hy5"
