File: VesselV2.kicad_pcb (KiCad board)
At the start: 2 copper layers, 345.3 x 176.2 mm, 220 parts, among them SW1 SW_Push, U1 ATmega32U4-A, Y1 16MHz

Commit message: Preliminary routing, Zone fill & DRC
Routing:
- net ROW5: track 0.00 -> 527.3 mm, vias 0 -> 3
- net ROW4: track 0.00 -> 496.4 mm, vias 0 -> 1
- net ROW2: track 0.00 -> 491.3 mm, vias 0 -> 1
- net ROW6: track 0.00 -> 470.2 mm, vias 0 -> 1
- net ROW3: track 0.00 -> 464.5 mm, vias 0 -> 1
- net COL0: track 0.00 -> 453.9 mm, vias 0 -> 1
- net COL1: track 0.00 -> 436.0 mm, vias 0 -> 2
- net ROW0: track 0.00 -> 433.6 mm, vias 0 -> 1
- net COL2: track 0.00 -> 421.7 mm, vias 0 -> 3
- net ROW1: track 0.00 -> 388.9 mm, vias 0 -> 4
- net COL3: track 0.00 -> 376.6 mm
- net COL4: track 0.00 -> 354.0 mm
- net COL5: track 0.00 -> 334.3 mm
- net COL6: track 0.00 -> 323.5 mm
- net COL7: track 0.00 -> 283.5 mm
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- added copper zone on B.Cu, net GND
- added copper zone on F.Cu, net GND

Commit message: Fixed routing errors - except USB footprint shape
Parts:
- S2: footprint PCM_marbastlib-mx:STAB_MX_P_2u -> PCM_marbastlib-mx:STAB_MX_P_ISO
- moved D61 2.38 mm to (372.3, 162.7)
- moved MX61 2.38 mm to (369.1, 161.9)
- moved S2 2.38 mm to (369.1, 161.9), turned to 0 degrees
Routing:
- net GND: track 249.2 -> 106.5 mm, vias 3 -> 12
- net ROW2: track 491.3 -> 462.2 mm
- net D+: track 156.3 -> 184.2 mm, vias 2 -> 0
- net ROW3: track 464.5 -> 490.2 mm
- net ROW5: track 527.3 -> 505.4 mm, vias 3 -> 1
- net ROW4: track 496.4 -> 474.7 mm
- net ROW6: track 470.2 -> 480.1 mm
- net ROW0: track 433.6 -> 441.8 mm
- net D-: track 153.2 -> 160.8 mm
- net COL2: track 421.7 -> 428.8 mm
- net COL6: track 323.5 -> 330.3 mm
- net ROW1: track 388.9 -> 382.2 mm
- net COL9: track 260.4 -> 266.6 mm
- net COL1: track 436.0 -> 440.8 mm
- net COL10: track 270.9 -> 275.4 mm
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
Commit message: Switch footprint swap - 3d models fixed - Routing (re)done - No errors other than USB footprint
Parts:
- MX1, MX10, MX100, MX101, MX102, MX11, MX12, MX13, MX14, MX15, MX16, MX17, MX18, MX19, MX2, MX20, MX21, MX22, MX23, MX24, MX25, MX26, MX27, MX28, MX29, MX3, MX30, MX31, MX32, MX33, MX34, MX35, MX36, MX37, MX38, MX39, MX4, MX40, MX41, MX42, MX43, MX44, MX46, MX47, MX49, MX5, MX50, MX51, MX52, MX53, MX54, MX55, MX56, MX57, MX58, MX59, MX6, MX60, MX62, MX63, MX65, MX66, MX67, MX68, MX69, MX7, MX70, MX71, MX72, MX73, MX74, MX75, MX76, MX77, MX78, MX8, MX80, MX81, MX82, MX83, MX84, MX85, MX86, MX87, MX88, MX89, MX9, MX90, MX92, MX93: footprint PCM_marbastlib-mx:SW_MX_1u -> PCM_Switch_Keyboard_Cherry_MX:SW_Cherry_MX_PCB_1.00u
- MX45: footprint PCM_marbastlib-mx:SW_MX_1u -> PCM_Switch_Keyboard_Cherry_MX:SW_Cherry_MX_PCB_2.00u
- MX48: footprint PCM_marbastlib-mx:SW_MX_1.5u -> PCM_Switch_Keyboard_Cherry_MX:SW_Cherry_MX_PCB_1.50u
- MX61: footprint PCM_marbastlib-mx:SW_MX_1u -> PCM_Switch_Keyboard_Cherry_MX:SW_Cherry_MX_PCB_ISOEnter
- MX64, MX91: footprint PCM_marbastlib-mx:SW_MX_1.75u -> PCM_Switch_Keyboard_Cherry_MX:SW_Cherry_MX_PCB_1.75u
- MX79, MX94, MX95, MX96, MX98, MX99: footprint PCM_marbastlib-mx:SW_MX_1.25u -> PCM_Switch_Keyboard_Cherry_MX:SW_Cherry_MX_PCB_1.25u
- MX97: footprint PCM_marbastlib-mx:SW_MX_1u -> PCM_Switch_Keyboard_Cherry_MX:SW_Cherry_MX_PCB_6.25u
- S1: footprint PCM_marbastlib-mx:STAB_MX_P_2u -> PCM_Mounting_Keyboard_Stabilizer:Stabilizer_Cherry_MX_2.00u
- S2: footprint PCM_marbastlib-mx:STAB_MX_P_ISO -> PCM_Mounting_Keyboard_Stabilizer:Stabilizer_Cherry_MX_2.00u
- S3: footprint PCM_marbastlib-mx:STAB_MX_P_6.25u -> PCM_Mounting_Keyboard_Stabilizer:Stabilizer_Cherry_MX_6.25u
- turned S1 to 0 degrees
- turned S2 to -90 degrees
Routing:
- net GND: track 106.5 -> 362.9 mm, vias 12 -> 13
- net ROW1: track 382.2 -> 449.7 mm, vias 4 -> 1
- net ROW0: track 441.8 -> 500.0 mm
- net COL1: track 440.8 -> 488.6 mm, vias 2 -> 0
- net ROW2: track 462.2 -> 420.8 mm
- net ROW3: track 490.2 -> 512.4 mm
- net D+: track 184.2 -> 164.3 mm, vias 0 -> 2
- net ROW5: track 505.4 -> 515.0 mm
- net ROW4: track 474.7 -> 467.6 mm, vias 1 -> 4
- net COL9: track 266.6 -> 260.5 mm
- net COL10: track 275.4 -> 269.3 mm
- net COL3: track 376.0 -> 381.9 mm, vias 0 -> 1
- net COL14: track 156.8 -> 151.9 mm, vias 0 -> 1
- net COL0: track 451.6 -> 456.4 mm
- net COL6: track 330.3 -> 333.9 mm
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